File: Electrical/Lights/Lights.sch (KiCad schematic (older format))
At the start: 39 parts

Commit message: single chip replacement start
Parts:
- added J? (x6): Conn_01x08_Male, symbol Connector:Conn_01x08_Male
- added J? (x6): Conn_01x01_Male, symbol Connector:Conn_01x01_Male
Connections:
- net labels added: V_USB
- wire segments 205 -> 329
