File: Electrical/Lights0.25/PowerManagment.sch (KiCad schematic (older format))
At the start: 35 parts

Commit message: pcb 0.25 rolled out
Parts:
- removed C?: .1uF, symbol Device:C
- removed R? (x2): R, symbol Device:R
- added C?: .1uF, symbol Device:C
- added R?: 50k, symbol Device:R
- added R?: 75k, symbol Device:R
- added R? (x2): 100k, symbol Device:R
- added R?: 200, symbol Device:R
- C?: value .1uF -> .03uF
- R1: value R -> 75k
- R2: value R -> 42.9k
- R3: value R -> 100k
- R4: value R -> 34.8k
- R? (x2): value R -> 39k
- R? (x2): value R -> 33k
- R?: value R -> 107k
- R?: value 42.6k -> 71k
- R?: value R -> 88k
- R?: value R -> NC
Connections:
- net labels added: +3V3, 3V3, NTC, USB_IN, VCC, VNTC, Vout
- net labels removed: +5V, ACOK, V_USB
- wire segments 101 -> 123
Other:
- note added: "Short press enables discharge mode\nLong press (>2.5s) disables discharge mode"
- note removed: "Short press enabled LED pins and disables after 5 sec\n"
